File: si-hardware-downled/si-hardware-downled.kicad_pcb (KiCad board)
At the start: 2 copper layers, 95 x 22.9 mm, 24 parts, among them U1 BP2866D, U2 S4525S

Commit message: export file gerber + drill
Parts:
- removed the ? at (160.5, 75.2)
- removed the ? at (170.1, 75.2)
- removed L1: 1mH, Inductor_SMD:L_Chilisin_BMRF00101040
- added FL1: 10mH, QSL_Filter:choke_4pin_7x8, F.Cu at (149.9, 82.9)
- added REF**: ESD-Logo_6.6x6mm_SilkScreen, Symbol:ESD-Logo_6.6x6mm_SilkScreen, F.Cu at (105.3, 68.4)
- added REF**: ESD-Logo_6.6x6mm_SilkScreen, Symbol:ESD-Logo_6.6x6mm_SilkScreen, F.Cu at (192.3, 84.9)
- added REF**: WEEE-Logo_4.2x6mm_SilkScreen, Symbol:WEEE-Logo_4.2x6mm_SilkScreen, F.Cu at (104.6, 84.9)
- C2: footprint Capacitor_THT:C_Radial_D5.0mm_H11.0mm_P2.00mm -> Capacitor_THT:C_Radial_D8.0mm_H11.5mm_P3.50mm
- C3: footprint Capacitor_THT:C_Radial_D5.0mm_H11.0mm_P2.00mm -> Capacitor_THT:C_Radial_D12.5mm_H20.0mm_P5.00mm
- moved C3 12.5 mm to (167.8, 79.1)
- moved R4 9.88 mm to (153.4, 85.5)
- moved D2 8.02 mm to (143.0, 83.6)
- moved R1 8.02 mm to (142.2, 69.7)
- moved U1 8.00 mm to (143.2, 77.0)
- moved R2 7.82 mm to (134.5, 69.8)
- moved C2 7.76 mm to (133.1, 78.0)
- moved D1 7.59 mm to (123.3, 76.6)
- moved R5 7.42 mm to (162.7, 85.5)
- moved D3 6.92 mm to (135.1, 83.6)
- moved C1 6.89 mm to (115.5, 76.5)
- moved F1 6.89 mm to (115.5, 70.6)
- moved R3 4.89 mm to (160.3, 68.2)
- moved ? 3.23 mm to (110.8, 68.5)
- moved ? 3.23 mm to (110.8, 83.9)
Connections:
- ? pad 2: Net-(J2-Pin_3) -> Net-(U2-D1-Pad7)
- ? pad 1: Net-(J1-Pin_1) -> unconnected-(F1-Pad1)
- ? pad 2: VCC -> VCC1
- ? pad 2: Net-(J2-Pin_2) -> Net-(U2-D2-Pad5)
- C3 pad 1: VCC -> VCC1
Routing:
- net Net-(U2-CLK): track 17.0 -> 20.8 mm
- net Net-(U1-ROVP): track 9.14 -> 10.5 mm
- net Net-(D2-A): track 10.2 -> 10.8 mm
- net Net-(U1-CS): track 12.4 -> 11.8 mm
- added copper zone on F.Cu, net VCC1
Other:
- board size 95 x 22.9 mm -> 95 x 23.5 mm
- board text added: "330VDC"

Commit message: change footprint
Parts:
- removed FL1: 10mH, QSL_Filter:choke_4pin_7x8
- added L1: 1mH/1A, Inductor_SMD:L_Coilcraft_MSS1210H-XXX, F.Cu at (157.2, 75.4)
- C1: footprint Capacitor_THT:C_Rect_L9.0mm_W3.4mm_P7.50mm_MKT -> Capacitor_THT:C_Rect_L11.0mm_W3.4mm_P10.00mm_MKT
- C3: value 22uF/400V -> 4.7uF/400V; footprint Capacitor_THT:C_Radial_D12.5mm_H20.0mm_P5.00mm -> Capacitor_THT:C_Radial_D8.0mm_H11.5mm_P3.50mm
- F1: value 500mA -> 500mA/250VAC; footprint Fuse:Fuse_1812_4532Metric -> SI_Fuse:Fuse_1808_4532Metric
- R1: value 180K -> 1R-1%; footprint Resistor_SMD:R_1206_3216Metric -> Resistor_SMD:R_1812_4532Metric
- R2: value 15K -> 18K
- moved R3 8.58 mm to (168.8, 67.1)
- moved F1 2.45 mm to (115.6, 68.2)
- moved C3 2.24 mm to (169.6, 77.7)
- moved ? 2.13 mm to (110.8, 86.1)
- moved R1 1.16 mm to (142.8, 68.8)
- turned ? to 90 degrees
Connections:
- ? pad 2: VCC1 -> VCC
- C3 pad 1: VCC1 -> VCC
Routing:
- net Net-(D2-A): track 10.8 -> 22.8 mm
- net Net-(U1-CS): track 11.8 -> 0.00 mm
- net Net-(U2-CLK): track 20.8 -> 14.6 mm
- added copper zone on F.Cu, net Net-(U1-CS)
- removed copper zone on B.Cu, net Net-(U2-D1-Pad7)
- removed copper zone on B.Cu, net Net-(U2-D2-Pad5)
- removed copper zone on F.Cu, net VCC1
Other:
- board text added: "+"
- board text added: "-"
- board text added: "12-36VDC"
- board text removed: "330VDC"
- board text removed: "L"

Commit message: final routing and placement
Parts:
- removed the REF** at (104.6, 84.9)
- moved REF** 18.5 mm to (123.9, 68.8)
- moved ? 6.60 mm to (179.8, 70.9)
- moved ? 6.60 mm to (179.8, 83.4)
- moved ? 6.60 mm to (179.8, 77.6)
- moved D3 6.60 mm to (128.5, 83.6)
- moved R5 6.60 mm to (156.1, 85.5)
- moved U2 6.60 mm to (172.3, 76.3)
- moved C3 6.60 mm to (163.0, 77.7)
- moved D2 6.60 mm to (136.4, 83.6)
- moved H2 6.60 mm to (186.0, 76.6)
- moved L1 6.60 mm to (150.6, 75.4)
- moved R1 6.60 mm to (136.2, 68.8)
- moved R3 6.60 mm to (162.2, 67.1)
- moved R4 6.60 mm to (146.8, 85.5)
- moved REF** 6.60 mm to (185.7, 84.9)
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Routing:
- net Net-(U1-ROVP): track 10.5 -> 8.89 mm
Other:
- board size 95 x 23.5 mm -> 88.4 x 23.5 mm
- board text added: "L"
